File: pcb/mini-one-pcb.kicad_pcb (KiCad board)
At the start: 4 copper layers, 50 x 70 mm, 119 parts, among them J1 ~{RUN}, J10 PYRO3, J11 MSD-1-A, J12 SMA_Edge, J13 SMA_Edge, J2 ~{SS}, J3 XT30-V-M, J4 USB1030, J5 PYRO1, J6 SERVO1, J7 SERVO2, J8 PYRO2, J9 PYRO ARM, Q1 AO3400A, Q2 AO3400A, Q3 AO3400A, U1 RP2354B, U2 AMS1117-3.3, U3 BMP585, U4 W25Q128JVSIQ, U5 LSM6DSV320XTR, U6 MAX-M10S, U7 RAK3172-8-SM-NI, Y1 ABM8-272-T3

Commit message: updates
Parts:
- added TP4: GND, TestPoint:TestPoint_Pad_D2.5mm, B.Cu at (139.9, 55.3)
- C34, C35, C40, C41, U3, U5: moved to F.Cu
- C36, C37, R23, R24, R25, U4: moved to B.Cu
- moved J12 113.0 mm to (106.0, 52.8), turned to 90 degrees
- moved J13 61.4 mm to (109.7, 116.7), turned to -90 degrees
- moved R26 60.1 mm to (54.8, 98.5), turned to 180 degrees
- moved R23 30.1 mm to (78.0, 68.9)
- moved C37 28.8 mm to (78.7, 66.0)
- moved C36 26.5 mm to (79.9, 66.0)
- moved R25 23.0 mm to (81.8, 66.5), turned to 0 degrees
- moved U4 19.8 mm to (83.5, 70.1), turned to 180 degrees
- moved R24 12.9 mm to (87.6, 66.8), turned to 0 degrees
- moved C35 10.4 mm to (105.6, 77.2), turned to 90 degrees
- moved C34 9.87 mm to (99.5, 77.2), turned to 90 degrees
- moved R21 9.50 mm to (101.0, 81.8), turned to 0 degrees
- moved U3 9.08 mm to (102.5, 77.6), turned to 90 degrees
- moved R22 8.58 mm to (103.0, 81.8), turned to 180 degrees
- moved R29 5.12 mm to (109.6, 80.8), turned to 0 degrees
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Connections:
- R5 pad 2: Net-(U1-GPIO20) -> Net-(U1-GPIO12)
- R6 pad 2: Net-(U1-GPIO21) -> Net-(U1-GPIO13)
- R7 pad 2: Net-(U1-GPIO22) -> Net-(U1-GPIO14)
- U1 pad 11: I2C_PIO_SDA -> Net-(U1-GPIO12)
- U1 pad 12: I2C_PIO_SCL -> Net-(U1-GPIO13)
- U1 pad 13: unconnected-(U1-GPIO14-Pad13) -> Net-(U1-GPIO14)
- U1 pad 20: Net-(U1-GPIO20) -> LoRA_~{RST}
- U1 pad 21: Net-(U1-GPIO21) -> unconnected-(U1-GPIO21-Pad21)
- U1 pad 22: Net-(U1-GPIO22) -> unconnected-(U1-GPIO22-Pad22)
- U1 pad 23: LoRA_~{RST} -> unconnected-(U1-GPIO23-Pad23)
- U1 pad 40: unconnected-(U1-GPIO32-Pad40) -> SERVO1_PWM
- U1 pad 45: SERVO1_PWM -> SERVO2_PWM
- U1 pad 46: SERVO2_PWM -> unconnected-(U1-GPIO37-Pad46)
- U1 pad 54: unconnected-(U1-GPIO43/ADC3-Pad54) -> PYRO1_GATE
- U1 pad 55: unconnected-(U1-GPIO44/ADC4-Pad55) -> PYRO2_GATE
- U1 pad 56: PYRO1_GATE -> PYRO3_GATE
- U1 pad 57: PYRO2_GATE -> unconnected-(U1-GPIO46/ADC6-Pad57)
- U1 pad 58: PYRO3_GATE -> unconnected-(U1-GPIO47/ADC7-Pad58)
Routing:
- net UART1_TX: track 37.3 -> 0.00 mm, vias 2 -> 0
- net UART1_RX: track 37.1 -> 0.00 mm, vias 2 -> 0
- net +1.1V: track 43.1 -> 8.30 mm, vias 1 -> 0
- net SPI0_MISO: track 29.9 -> 0.00 mm
- net SPI0_~{CS}: track 29.8 -> 0.00 mm, vias 2 -> 0
- net SPI1_MISO: track 28.2 -> 0.00 mm, vias 1 -> 0
- net SERVO1_PWM: track 27.5 -> 0.00 mm
- net SPI1_SCK: track 27.4 -> 0.00 mm, vias 1 -> 0
- net SPI1_MOSI: track 26.6 -> 0.00 mm, vias 1 -> 0
- net USB_D+: track 25.8 -> 0.00 mm, vias 1 -> 0
- net SPI1_~{CS}: track 24.7 -> 0.00 mm, vias 1 -> 0
- net USB_D-: track 22.7 -> 0.00 mm, vias 1 -> 0
- net SPI0_SCK: track 22.2 -> 0.00 mm
- net SERVO2_PWM: track 21.9 -> 0.00 mm
- net Net-(U1-GPIO20): track 20.3 -> 0.00 mm
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Other:
- outline, holes or cut-outs redrawn
- board text added: "- + S"
- board text added: "1V1"
- board text added: "2S LIPO IN"
- board text added: "3V3"
- board text added: "A"
- board text added: "B"
- board text added: "C"
- board text added: "PYRO 1"
- board text added: "PYRO 2"
- board text added: "PYRO 3"
- board text added: "PYRO EN"
- board text added: "RP2354B"
- board text added: "RUN"
- board text added: "SENSORS"
- board text added: "SERVO 1"
- board text added: "SERVO 2"
- board text added: "~{SS}"
