File: pcb/mini-one-pcb.kicad_pcb (KiCad board)
At the start: 4 copper layers, 50 x 70 mm, 120 parts, among them J1 ~{RUN}, J10 PYRO3, J11 MSD-1-A, J12 SMA_Edge, J13 SMA_Edge, J2 ~{SS}, J3 XT30-V-M, J4 USB1030, J5 PYRO1, J6 SERVO1, J7 SERVO2, J8 PYRO2, J9 PYRO ARM, Q1 AO3400A, Q2 AO3400A, Q3 AO3400A, U1 RP2354B, U2 AMS1117-3.3, U3 BMP585, U4 W25Q128JVSIQ, U5 LSM6DSV320XTR, U6 MAX-M10S, U7 RAK3172-8-SM-NI, Y1 ABM8-272-T3

Commit message: PCB update
Parts:
- moved R26 60.0 mm to (114.8, 101.4), turned to -90 degrees
- moved C36 29.2 mm to (100.3, 86.9)
- moved C37 29.2 mm to (99.1, 86.9)
- moved R23 29.2 mm to (98.4, 89.8)
- moved R25 29.2 mm to (102.2, 87.4)
- moved U4 29.2 mm to (103.9, 91.0)
- moved R24 28.9 mm to (108.0, 87.2)
- moved C17 2.42 mm to (113.3, 78.9)
- moved R28 2.15 mm to (111.9, 100.9), turned to 180 degrees
- moved R30 2.08 mm to (109.6, 80.6), turned to 0 degrees
- moved R29 2.07 mm to (111.7, 80.6), turned to 180 degrees
- moved TP2 0.39 mm to (136.3, 55.3)
- moved TP1 0.39 mm to (128.1, 55.3)
- moved TP3 0.39 mm to (132.3, 55.3)
- moved TP4 0.39 mm to (140.3, 55.3)
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Connections:
- U1 pad 2: +3.3V -> unconnected-(U1-GPIO5-Pad2)
- U1 pad 3: +3.3V -> unconnected-(U1-GPIO6-Pad3)
Routing:
- net UART1_TX: track 0.00 -> 28.1 mm, vias 0 -> 2
- net UART1_RX: track 0.00 -> 27.7 mm, vias 0 -> 2
- net SPI1_SCK: track 0.00 -> 27.2 mm, vias 0 -> 1
- net SPI1_MISO: track 0.00 -> 25.7 mm, vias 0 -> 1
- net SPI1_MOSI: track 0.00 -> 25.7 mm, vias 0 -> 1
- net SPI1_~{CS}: track 0.00 -> 24.0 mm, vias 0 -> 1
- net USB_D+: track 0.00 -> 23.6 mm, vias 0 -> 1
- net SERVO2_PWM: track 0.00 -> 22.4 mm
- net +1.1V: track 8.30 -> 30.5 mm, vias 0 -> 1
- net USB_D-: track 0.00 -> 20.5 mm, vias 0 -> 1
- net SERVO1_PWM: track 0.00 -> 20.4 mm
- net SPI0_MOSI: track 0.00 -> 17.3 mm, vias 0 -> 1
- net SPI0_SCK: track 0.00 -> 16.4 mm, vias 0 -> 1
- net GNSS_~{RST}: track 2.98 -> 19.1 mm, vias 0 -> 2
- net LoRA_~{RST}: track 2.48 -> 18.1 mm
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Other:
- board text added: "12 MHz"
- board text added: "16 MB"
- board text added: "2S LiFe IN"
- board text added: "5V0"
- board text added: "Edward S. 2026"
- board text added: "GND"
- board text added: "GNSS"
- board text added: "LoRa"
- board text added: "MEMORY"
- board text added: "PY EN"
- board text added: "TEST POINTS"
- board text added: "WARNING Do not power the board without any antennas connected!"
- board text removed: "2S LIPO IN"
- board text removed: "PYRO EN"
