File: pcb/RF.kicad_sch (KiCad schematic)
At the start: 13 parts, among them J12 SMA_Edge, J13 SMA_Edge, U6 MAX-M10S, U7 RAK3172-8-SM-NI

Commit message: PCB update
Parts:
- J12, J13, TP3: now not fitted
Changed lines of the file:
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@@
 		(on_board yes)
 		(in_pos_files yes)
-		(dnp no)
+		(dnp yes)
 		(fields_autoplaced yes)
 		(property "Reference" "J13"
@@
 		(on_board yes)
 		(in_pos_files yes)
-		(dnp no)
+		(dnp yes)
 		(fields_autoplaced yes)
 		(property "Reference" "J12"
@@
 		(on_board yes)
 		(in_pos_files yes)
-		(dnp no)
+		(dnp yes)
 		(property "Reference" "TP3"
 			(at 171.323 184.277 90)
