File: pcb/processor.kicad_sch (KiCad schematic)
At the start: 38 parts, among them J1 ~{RUN}, J2 ~{SS}, U1 RP2354B, Y1 ABM8-272-T3

Commit message: updates
Connections:
- net I2C_PIO_SCL is gone; now on an unnamed net: U1.12 (GPIO13)
- net I2C_PIO_SDA is gone; now on an unnamed net: U1.11 (GPIO12)
- net LoRA_~{RST}: now also U1.20 (GPIO20); no longer U1.23 (GPIO23)
- net PYRO1_GATE: now also U1.54 (GPIO43/ADC3); no longer U1.56 (GPIO45/ADC5)
- net PYRO2_GATE: now also U1.55 (GPIO44/ADC4); no longer U1.57 (GPIO46/ADC6)
- net PYRO3_GATE: now also U1.56 (GPIO45/ADC5); no longer U1.58 (GPIO47/ADC7)
- net SERVO1_PWM: now also U1.40 (GPIO32); no longer U1.45 (GPIO36)
- net SERVO2_PWM: now also U1.45 (GPIO36); no longer U1.46 (GPIO37)
- net at R7.2: now also U1.13 (GPIO14); no longer U1.22 (GPIO22)
- net at R5.2: no longer U1.20 (GPIO20)
- net at R6.2: no longer U1.21 (GPIO21)
- no-connect marks 24 -> 26
Other:
- moved on the sheet: D1, D2, D3, R5, R6, R7

Commit message: PCB update
Parts:
- J1, J2, TP1: now not fitted
Connections:
- net +3.3V: no longer U1.2 (GPIO5), U1.3 (GPIO6)
- no-connect marks 26 -> 28
Other:
- note removed: "Tied HIGH for routing purposes; set the GPIO to high-impedance"
Changed lines of the file:
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@@
 		)
 	)
-	(text "Tied HIGH for routing purposes; set the GPIO to high-impedance"
-		(exclude_from_sim no)
-		(at 138.938 83.312 0)
-		(effects
-			(font
-				(size 1.27 1.27)
-			)
-		)
-	)
 	(text "Decoupling capacitors, Keep close to MCU (<2mm)"
 		(exclude_from_sim no)
@@
 	)
 	(junction
-		(at 102.87 81.28)
-		(diameter 0)
-		(color 0 0 0 0)
-	)
-	(junction
 		(at 213.36 87.63)
 		(diameter 0)
@@
 	)
 	(no_connect
+		(at 101.6 83.82)
+	)
+	(no_connect
 		(at 101.6 127)
 	)
@@
 	)
 	(no_connect
+		(at 101.6 81.28)
+	)
+	(no_connect
 		(at 50.8 109.22)
 	)
@@
 	(wire
 		(pts
-			(xy 101.6 81.28) (xy 102.87 81.28)
-		)
-		(stroke
-			(width 0)
-			(type default)
-		)
-	)
-	(wire
-		(pts
 			(xy 76.2 177.8) (xy 76.2 176.53)
 		)
@@
 	(wire
 		(pts
-			(xy 102.87 81.28) (xy 116.84 81.28)
-		)
-		(stroke
-			(width 0)
-			(type default)
-		)
-	)
-	(wire
-		(pts
 			(xy 214.63 49.53) (xy 227.33 49.53)
 		)
@@
 	(wire
 		(pts
-			(xy 116.84 80.01) (xy 116.84 81.28)
-		)
-		(stroke
-			(width 0)
-			(type default)
-		)
-	)
-	(wire
-		(pts
 			(xy 240.03 148.59) (xy 240.03 146.05)
 		)
@@
 	(wire
 		(pts
-			(xy 102.87 81.28) (xy 102.87 83.82)
-		)
-		(stroke
-			(width 0)
-			(type default)
-		)
-	)
-	(wire
-		(pts
 			(xy 137.16 104.14) (xy 146.05 104.14)
 		)
@@
 	(wire
 		(pts
-			(xy 102.87 83.82) (xy 101.6 83.82)
-		)
-		(stroke
-			(width 0)
-			(type default)
-		)
-	)
-	(wire
-		(pts
 			(xy 209.55 31.75) (xy 220.98 31.75)
 		)
@@
 	(symbol
 		(lib_id "power:+3.3V")
-		(at 116.84 80.01 0)
-		(unit 1)
-		(body_style 1)
-		(exclude_from_sim no)
-		(in_bom yes)
-		(on_board yes)
-		(in_pos_files yes)
-		(dnp no)
-		(property "Reference" "#PWR09"
-			(at 116.84 83.82 0)
-			(hide yes)
-			(show_name no)
-			(do_not_autoplace no)
-			(effects
-				(font
-					(size 1.27 1.27)
-				)
-			)
-		)
-		(property "Value" "+3.3V"
-			(at 116.84 76.2 0)
-			(show_name no)
-			(do_not_autoplace no)
-			(effects
-				(font
-					(size 1.27 1.27)
-				)
-			)
-		)
-		(property "Footprint" ""
-			(at 116.84 80.01 0)
-			(hide yes)
-			(show_name no)
-			(do_not_autoplace no)
-			(effects
-				(font
-					(size 1.27 1.27)
-				)
-			)
-		)
-		(property "Datasheet" ""
-			(at 116.84 80.01 0)
-			(hide yes)
-			(show_name no)
-			(do_not_autoplace no)
-			(effects
-				(font
-					(size 1.27 1.27)
-				)
-			)
-		)
-		(property "Description" "Power symbol creates a global label with name \"+3.3V\""
-			(at 116.84 80.01 0)
-			(hide yes)
-			(show_name no)
-			(do_not_autoplace no)
-			(effects
-				(font
-					(size 1.27 1.27)
-				)
-			)
-		)
-		(pin "1"
-		)
-		(instances
-			(project "mini-one-pcb"
-				(path "/ceb43049-5cbf-4c56-aa0a-c2184d7e2ca1/f3daba49-5080-4654-9217-67c35ea0f53f"
-					(reference "#PWR09")
-					(unit 1)
-				)
-			)
-		)
-	)
-	(symbol
-		(lib_id "power:+3.3V")
 		(at 186.69 22.86 0)
 		(unit 1)
@@
 		(on_board yes)
 		(in_pos_files yes)
-		(dnp no)
+		(dnp yes)
 		(property "Reference" "J2"
 			(at 44.958 109.474 90)
@@
 		(on_board yes)
 		(in_pos_files yes)
-		(dnp no)
+		(dnp yes)
 		(property "Reference" "J1"
 			(at 42.418 76.2 90)
@@
 		(on_board yes)
 		(in_pos_files yes)
-		(dnp no)
+		(dnp yes)
 		(property "Reference" "TP1"
 			(at 278.13 82.55 90)
